Commit message: style: add spacers to urdf

File: description/robot_core.xacro (robot description, xacro)
@@ -41,5 +41,29 @@
             <material name="white"/>
         </visual>
-        <!--  -->
+        <!-- Spacers -->
+        <visual>
+            <origin xyz="0.060 0.033 0.085"/>
+            <geometry>
+                <cylinder radius="0.002" length="0.125"/>
+            </geometry>
+        </visual>
+        <visual>
+            <origin xyz="0.060 -0.033 0.085"/>
+            <geometry>
+                <cylinder radius="0.002" length="0.125"/>
+            </geometry>
+        </visual>
+        <visual>
+            <origin xyz="-0.060 0.033 0.085"/>
+            <geometry>
+                <cylinder radius="0.002" length="0.125"/>
+            </geometry>
+        </visual>
+        <visual>
+            <origin xyz="-0.060 -0.033 0.085"/>
+            <geometry>
+                <cylinder radius="0.002" length="0.125"/>
+            </geometry>
+        </visual>
         <!-- front free wheel -->
         <visual>

Commit message: feat: add collision and inertial boxes

File: description/robot_core.xacro (robot description, xacro)
@@ -3,4 +3,5 @@
     <!-- Include the colors file -->
     <xacro:include filename="$(find slambot)/description/colors.xacro"/>
+    <xacro:include filename="$(find slambot)/description/inertial_macros.xacro"/>
     <!-- Base link -->
     <link name="base_link"></link>
@@ -94,4 +95,14 @@
             <material name="white"/>
         </visual>
+        <collision>
+            <origin xyz="0 0 0.100"/>
+            <geometry>
+                <cylinder radius="0.08" length="0.200"/>
+            </geometry>
+            <material name="white"/>
+        </collision>
+        <xacro:inertial_cylinder mass="1.0" radius="0.08" length="0.200">
+            <origin xyz="0 0 0.100" rpy="0 0 0"/>
+        </xacro:inertial_cylinder>
     </link>
     <!-- Left Wheel -->

Commit message: refactor: split robot_core.xacro code

File: description/robot_core.xacro (robot description, xacro)
@@ -1,209 +1,14 @@
 <?xml version="1.0"?>
 <robot xmlns:xacro="http://www.ros.org/wiki/xacro">
-    <!-- Include the colors file -->
     <xacro:include filename="$(find slambot)/description/colors.xacro"/>
     <xacro:include filename="$(find slambot)/description/inertial_macros.xacro"/>
-    <!-- Base link -->
-    <link name="base_link"></link>
-    <!-- Chassis link -->
-    <joint name="chassis_joint" type="fixed">
-        <parent link="base_link"/>
-        <child link="chassis"/>
-        <origin xyz="0 0 0"/>
-    </joint>
-    <link name="chassis">
-        <!-- Levels -->
-        <visual>
-            <origin xyz="0 0 0.020"/>
-            <geometry>
-                <box size="0.14 0.10 0.01"/>
-            </geometry>
-            <material name="white"/>
-        </visual>
-        <visual>
-            <origin xyz="0 0 0.070"/>
-            <geometry>
-                <cylinder radius="0.08" length="0.01"/>
-            </geometry>
-            <material name="white"/>
-        </visual>
-        <visual>
-            <origin xyz="0 0 0.120"/>
-            <geometry>
-                <cylinder radius="0.08" length="0.01"/>
-            </geometry>
-            <material name="white"/>
-        </visual>
-        <visual>
-            <origin xyz="0 0 0.150"/>
-            <geometry>
-                <box size="0.125 0.075 0.01"/>
-            </geometry>
-            <material name="white"/>
-        </visual>
-        <!-- Spacers -->
-        <visual>
-            <origin xyz="0.060 0.033 0.085"/>
-            <geometry>
-                <cylinder radius="0.002" length="0.125"/>
-            </geometry>
-        </visual>
-        <visual>
-            <origin xyz="0.060 -0.033 0.085"/>
-            <geometry>
-                <cylinder radius="0.002" length="0.125"/>
-            </geometry>
-        </visual>
-        <visual>
-            <origin xyz="-0.060 0.033 0.085"/>
-            <geometry>
-                <cylinder radius="0.002" length="0.125"/>
-            </geometry>
-        </visual>
-        <visual>
-            <origin xyz="-0.060 -0.033 0.085"/>
-            <geometry>
-                <cylinder radius="0.002" length="0.125"/>
-            </geometry>
-        </visual>
-        <!-- front free wheel -->
-        <visual>
-            <origin xyz="0.045 0 0"/>
-            <geometry>
-                <cylinder radius="0.015" length="0.030"/>
-            </geometry>
-        </visual>
-        <visual>
-            <origin xyz="0.045 0 -0.015"/>
-            <geometry>
-                <sphere radius="0.015"/>
-            </geometry>
-            <material name="white"/>
-        </visual>
-        <!-- back free wheel -->
-        <visual>
-            <origin xyz="-0.045 0 0"/>
-            <geometry>
-                <cylinder radius="0.015" length="0.030"/>
-            </geometry>
-        </visual>
-        <visual>
-            <origin xyz="-0.045 0 -0.015"/>
-            <geometry>
-                <sphere radius="0.015"/>
-            </geometry>
-            <material name="white"/>
-        </visual>
-        <collision>
-            <origin xyz="0 0 0.100"/>
-            <geometry>
-                <cylinder radius="0.08" length="0.200"/>
-            </geometry>
-            <material name="white"/>
-        </collision>
-        <xacro:inertial_cylinder mass="1.0" radius="0.08" length="0.200">
-            <origin xyz="0 0 0.100" rpy="0 0 0"/>
-        </xacro:inertial_cylinder>
-    </link>
-    <!-- Left Wheel -->
-    <!-- Wheel -->
-    <joint name="left_wheel_joint" type="continuous">
-        <parent link="base_link"/>
-        <child link="left_wheel"/>
-        <origin xyz="0 0.065 0" rpy="-${pi/2} 0 0"/>
-        <axis xyz="0 0 1"/>
-    </joint>
-    <link name="left_wheel">
-        <visual>
-            <geometry>
-                <cylinder radius="0.035" length="0.0249"/>
-            </geometry>
-            <material name="black"/>
-        </visual>
-    </link>
-    <!-- Tire -->
-    <joint name="left_tire_joint" type="fixed">
-        <parent link="left_wheel"/>
-        <child link="left_tire"/>
-    </joint>
-    <link name="left_tire">
-        <visual>
-            <geometry>
-                <cylinder radius="0.025" length="0.0250"/>
-            </geometry>
-            <material name="yellow"/>
-        </visual>
-    </link>
-    <!-- Right Wheel -->
-    <!-- Wheel -->
-    <joint name="right_wheel_joint" type="continuous">
-        <parent link="base_link"/>
-        <child link="right_wheel"/>
-        <origin xyz="0 -0.065 0" rpy="-${pi/2} 0 0"/>
-        <axis xyz="0 0 1"/>
-    </joint>
-    <link name="right_wheel">
-        <visual>
-            <geometry>
-                <cylinder radius="0.035" length="0.0249"/>
-            </geometry>
-            <material name="black"/>
-        </visual>
-    </link>
-    <!-- Tire -->
-    <joint name="right_tire_joint" type="fixed">
-        <parent link="right_wheel"/>
-        <child link="right_tire"/>
-    </joint>
-    <link name="right_tire">
-        <visual>
-            <geometry>
-                <cylinder radius="0.025" length="0.0250"/>
-            </geometry>
-            <material name="yellow"/>
-        </visual>
-    </link>
-    <!-- LIDAR -->
-    <joint name="lidar_joint" type="fixed">
-        <parent link="base_link"/>
-        <child link="lidar"/>
-        <origin xyz="0.02 0 0.185" rpy="0 0 0"/>
-    </joint>
-    <link name="lidar">
-        <visual>
-            <origin xyz="0 0 -0.020"/>
-            <geometry>
-                <box size="0.055 0.055 0.025"/>
-            </geometry>
-            <material name="black"/>
-        </visual>
-        <visual>
-            <origin xyz="0 0 -0.0125"/>
-            <geometry>
-                <cylinder radius="0.026" length="0.040"/>
-            </geometry>
-            <material name="black"/>
-        </visual>
-    </link>
-    <!-- Camera -->
-    <joint name="cam_joint" type="fixed">
-        <parent link="base_link"/>
-        <child link="cam"/>
-        <origin xyz="0.07 0 0.135" rpy="0 ${pi/2} 0"/>
-    </joint>
-    <link name="cam">
-        <visual>
-            <origin xyz="0 0 -0.01"/>
-            <geometry>
-                <box size="0.020 0.020 0.010"/>
-            </geometry>
-            <material name="black"/>
-        </visual>
-        <visual>
-            <geometry>
-                <cylinder radius="0.006" length="0.010"/>
-            </geometry>
-            <material name="black"/>
-        </visual>
-    </link>
+    <xacro:include filename="$(find slambot)/description/chassis.xacro"/>
+    <xacro:include filename="$(find slambot)/description/wheel.xacro"/>
+    <xacro:include filename="$(find slambot)/description/sensors.xacro"/>
+    <link name="base_link"/>
+    <xacro:chassis_body/>
+    <xacro:drive_wheel side="left" y_offset="0.065"/>
+    <xacro:drive_wheel side="right" y_offset="-0.065"/>
+    <xacro:lidar_sensor/>
+    <xacro:camera_sensor/>
 </robot>
